File: metrocard.kicad_pcb (KiCad board)
At the start: 2 copper layers, 85 x 53 mm, 65 parts, among them J1 Conn_01x04, U1 HT16K33A-24SOP

Commit message: added readme
Parts:
- J1: footprint Connector_JST:JST_EH_B4B-EH-A_1x04_P2.50mm_Vertical -> Connector_PinHeader_2.54mm:PinHeader_1x04_P2.54mm_Vertical
- turned J1 to 180 degrees
Routing:
- net R3: track 128.2 -> 128.9 mm
Changed lines of the file:
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@@
 			(drillshape 0)
 			(scaleselection 1)
-			(outputdirectory "../../metrocard_pone_g/")
+			(outputdirectory "../metrocard_module_ger0.1/")
 		)
 	)
@@
 		(embedded_fonts no)
 	)
-	(footprint "Connector_JST:JST_EH_B4B-EH-A_1x04_P2.50mm_Vertical"
+	(footprint "Connector_PinHeader_2.54mm:PinHeader_1x04_P2.54mm_Vertical"
 		(layer "F.Cu")
-		(at 233.45 100.46 90)
-		(descr "JST EH series connector, B4B-EH-A (http://www.jst-mfg.com/product/pdf/eng/eEH.pdf), generated with kicad-footprint-generator")
-		(tags "connector JST EH vertical")
+		(at 233.45 100.46 180)
+		(descr "Through hole straight pin header, 1x04, 2.54mm pitch, single row")
+		(tags "Through hole pin header THT 1x04 2.54mm single row")
 		(property "Reference" "J1"
-			(at 3.749999 -2.8 90)
-			(layer "F.Fab")
+			(at 0 -2.38 0)
+			(layer "F.SilkS")
 			(effects
 				(font
@@
 		)
 		(property "Value" "Conn_01x04"
-			(at 3.749999 3.4 90)
+			(at 0 10 0)
 			(layer "F.Fab")
 			(effects
@@
 			)
 		)
-		(property "Datasheet" "~"
-			(at 0 0 90)
+		(property "Datasheet" ""
+			(at 0 0 0)
 			(layer "F.Fab")
 			(hide yes)
@@
 			)
 		)
-		(property "Description" "Generic connector, single row, 01x04, script generated (kicad-library-utils/schlib/autogen/connector/)"
-			(at 0 0 90)
+		(property "Description" ""
+			(at 0 0 0)
 			(layer "F.Fab")
 			(hide yes)
@@
 		(attr through_hole)
 		(fp_line
-			(start 9.61 -1.21)
-			(end 9.61 0)
-			(stroke
-				(width 0.12)
-				(type solid)
-			)
-			(layer "F.SilkS")
-		)
-		(fp_line
-			(start -2.11 -1.21)
-			(end 9.61 -1.21)
+			(start 1.38 1.27)
+			(end 1.379999 9)
 			(stroke
 				(width 0.12)
@@
 		)
 		(fp_line
-			(start 9.61 0)
-			(end 10.110001 0)
+			(start -1.379999 9)
+			(end 1.379999 9)
 			(stroke
 				(width 0.12)
@@
 		)
 		(fp_line
-			(start -2.11 0)
-			(end -2.11 -1.21)
+			(start -1.379999 0)
+			(end -1.38 -1.38)
 			(stroke
 				(width 0.12)
@@
 		)
 		(fp_line
-			(start -2.61 0)
-			(end -2.11 0)
+			(start -1.38 1.27)
+			(end 1.38 1.27)
 			(stroke
 				(width 0.12)
@@
 		)
 		(fp_line
-			(start -2.91 0.11)
-			(end -2.91 2.61)
+			(start -1.38 1.27)
+			(end -1.379999 9)
 			(stroke
 				(width 0.12)
@@
 		)
 		(fp_line
-			(start 10.11 0.81)
-			(end 9.11 0.81)
+			(start -1.38 -1.38)
+			(end 0 -1.379999)
 			(stroke
 				(width 0.12)
@@
 			(layer "F.SilkS")
 		)
-		(fp_line
-			(start 9.11 0.81)
-			(end 9.11 2.31)
-			(stroke
-				(width 0.12)
-				(type solid)
+		(fp_poly
+			(pts
+				(xy -1.77 -1.77) (xy -1.77 9.39) (xy 1.77 9.39) (xy 1.77 -1.77)
 			)
-			(layer "F.SilkS")
-		)
-		(fp_line
-			(start -1.609999 0.81)
-			(end -1.61 2.31)
 			(stroke
-				(width 0.12)
+				(width 0.05)
 				(type solid)
 			)
-			(layer "F.SilkS")
+			(fill no)
+			(layer "F.CrtYd")
 		)
 		(fp_line
-			(start -2.61 0.81)
-			(end -1.609999 0.81)
+			(start 1.27 8.89)
+			(end -1.27 8.89)
 			(stroke
-				(width 0.12)
+				(width 0.1)
 				(type solid)
 			)
-			(layer "F.SilkS")
+			(layer "F.Fab")
 		)
 		(fp_line
-			(start -2.91 2.61)
-			(end -0.41 2.61)
-			(stroke
-				(width 0.12)
-				(type solid)
-			)
-			(layer "F.SilkS")
-		)
-		(fp_poly
-			(pts
-				(xy -2.61 -1.71) (xy 10.11 -1.71) (xy 10.11 2.31) (xy -2.61 2.31)
-			)
+			(start 1.27 -1.27)
+			(end 1.27 8.89)
 			(stroke
-				(width 0.12)
-				(type solid)
-			)
-			(fill no)
-			(layer "F.SilkS")
-		)
-		(fp_poly
-			(pts
-				(xy -3 -2.1) (xy 10.5 -2.1) (xy 10.5 2.7) (xy -3 2.7)
-			)
-			(stroke
-				(width 0.05)
+				(width 0.1)
 				(type solid)
 			)
-			(fill no)
-			(layer "F.CrtYd")
+			(layer "F.Fab")
 		)
 		(fp_line
-			(start -2.91 0.11)
-			(end -2.91 2.61)
+			(start -0.635 -1.27)
+			(end 1.27 -1.27)
 			(stroke
 				(width 0.1)
@@
 		)
 		(fp_line
-			(start -2.91 2.61)
-			(end -0.41 2.61)
+			(start -1.27 8.89)
+			(end -1.27 -0.635)
 			(stroke
 				(width 0.1)
@@
 			(layer "F.Fab")
 		)
-		(fp_poly
-			(pts
-				(xy -2.5 -1.6) (xy 10 -1.6) (xy 10 2.2) (xy -2.5 2.2)
-			)
+		(fp_line
+			(start -1.27 -0.635)
+			(end -0.635 -1.27)
 			(stroke
 				(width 0.1)
 				(type solid)
 			)
-			(fill no)
 			(layer "F.Fab")
 		)
 		(fp_text user "${REFERENCE}"
-			(at 3.75 1.5 90)
+			(at 0 3.81 90)
 			(layer "F.Fab")
 			(effects
@@
 			)
 		)
-		(pad "1" thru_hole roundrect
-			(at 0 0 90)
-			(size 1.7 1.95)
-			(drill 0.95)
+		(pad "1" thru_hole rect
+			(at 0 0 180)
+			(size 1.7 1.7)
+			(drill 1)
 			(layers "*.Cu" "*.Mask")
 			(remove_unused_layers no)
-			(roundrect_rratio 0.147059)
 			(net 18 "SCL")
 			(pinfunction "Pin_1")
 			(pintype "passive")
 		)
-		(pad "2" thru_hole oval
-			(at 2.5 0 90)
-			(size 1.7 1.95)
-			(drill 0.95)
+		(pad "2" thru_hole circle
+			(at 0 2.54 180)
+			(size 1.7 1.7)
+			(drill 1)
 			(layers "*.Cu" "*.Mask")
 			(remove_unused_layers no)
@@
 			(pintype "passive")
 		)
-		(pad "3" thru_hole oval
-			(at 5 0 90)
-			(size 1.7 1.95)
-			(drill 0.95)
+		(pad "3" thru_hole circle
+			(at 0 5.079999 180)
+			(size 1.7 1.7)
+			(drill 1)
 			(layers "*.Cu" "*.Mask")
 			(remove_unused_layers no)
@@
 			(pintype "passive")
 		)
-		(pad "4" thru_hole oval
-			(at 7.5 0 90)
-			(size 1.7 1.95)
-			(drill 0.95)
+		(pad "4" thru_hole circle
+			(at 0 7.62 180)
+			(size 1.7 1.7)
+			(drill 1)
 			(layers "*.Cu" "*.Mask")
 			(remove_unused_layers no)
@@
 		)
 		(embedded_fonts no)
-		(model "${KICAD9_3DMODEL_DIR}/Connector_JST.3dshapes/JST_EH_B4B-EH-A_1x04_P2.50mm_Vertical.step"
+		(model "${KICAD9_3DMODEL_DIR}/Connector_PinHeader_2.54mm.3dshapes/PinHeader_1x04_P2.54mm_Vertical.step"
 			(offset
 				(xyz 0 0 0)
@@
 	)
 	(segment
-		(start 222.638528 88.8)
-		(end 227.673221 88.8)
+		(start 169.98 86.670001)
+		(end 169.96 86.690001)
 		(width 0.4)
 		(layer "F.Cu")
@@
 	)
 	(segment
-		(start 231.2 85.273221)
-		(end 231.2 73.611472)
+		(start 188.02 81.670001)
+		(end 187.76 81.930001)
 		(width 0.4)
 		(layer "F.Cu")
@@
 	)
 	(segment
-		(start 169.98 86.670001)
-		(end 169.96 86.690001)
+		(start 230.01 71.25)
+		(end 192.37 71.25)
 		(width 0.4)
 		(layer "F.Cu")
@@
 	)
 	(segment
-		(start 188.02 81.670001)
-		(end 187.76 81.930001)
+		(start 231.25 85.293931)
+		(end 231.25 73.590761)
 		(width 0.4)
 		(layer "F.Cu")
@@
 	)
 	(segment
-		(start 220.188528 91.25)
-		(end 222.638528 88.8)
+		(start 220.278528 91.16)
+		(end 220.349239 91.16)
 		(width 0.4)
 		(layer "F.Cu")
@@
 	)
 	(segment
+		(start 220.349239 91.16)
+		(end 222.659238 88.85)
+		(width 0.4)
+		(layer "F.Cu")
+		(net 13)
+	)
+	(segment
 		(start 187.76 81.930001)
 		(end 186.77 81.930001)
@@
 	)
 	(segment
-		(start 186.77 81.930001)
-		(end 184.43 84.270001)
+		(start 212.25708 94.04)
+		(end 212.25708 92.58292)
 		(width 0.4)
 		(layer "F.Cu")
@@
 	)
 	(segment
-		(start 228.838528 71.25)
-		(end 192.37 71.25)
+		(start 186.77 81.930001)
+		(end 184.43 84.270001)
 		(width 0.4)
 		(layer "F.Cu")
@@
 	)
 	(segment
-		(start 213.59 91.25)
-		(end 220.188528 91.25)
+		(start 231.25 73.590761)
+		(end 231.24 73.580761)
 		(width 0.4)
 		(layer "F.Cu")
@@
 	)
 	(segment
-		(start 183.699999 84.270001)
-		(end 181.279999 86.690001)
+		(start 222.659238 88.85)
+		(end 227.693931 88.85)
 		(width 0.4)
 		(layer "F.Cu")
@@
 	)
 	(segment
-		(start 212.25708 92.58292)
-		(end 213.59 91.25)
+		(start 183.699999 84.270001)
+		(end 181.279999 86.690001)
 		(width 0.4)
 		(layer "F.Cu")
@@
 	)
 	(segment
-		(start 231.2 73.611472)
-		(end 228.838528 71.25)
+		(start 174.52 86.690001)
+		(end 174.5 86.670001)
 		(width 0.4)
 		(layer "F.Cu")
@@
 	)
 	(segment
-		(start 174.52 86.690001)
-		(end 174.5 86.670001)
+		(start 212.25708 92.58292)
+		(end 213.59 91.25)
 		(width 0.4)
 		(layer "F.Cu")
@@
 	)
 	(segment
-		(start 227.673221 88.8)
-		(end 231.2 85.273221)
+		(start 231.24 72.48)
+		(end 230.01 71.25)
 		(width 0.4)
 		(layer "F.Cu")
@@
 	)
 	(segment
+		(start 213.59 91.25)
+		(end 220.188528 91.25)
+		(width 0.4)
+		(layer "F.Cu")
+		(net 13)
+	)
+	(segment
 		(start 169.96 86.690001)
 		(end 169.570001 86.690001)
@@
 	)
 	(segment
+		(start 220.188528 91.25)
+		(end 220.278528 91.16)
+		(width 0.4)
+		(layer "F.Cu")
+		(net 13)
+	)
+	(segment
+		(start 231.24 73.580761)
+		(end 231.24 72.48)
+		(width 0.4)
+		(layer "F.Cu")
+		(net 13)
+	)
+	(segment
 		(start 179.579998 86.690001)
 		(end 174.52 86.690001)
@@
 	)
 	(segment
-		(start 212.25708 94.04)
-		(end 212.25708 92.58292)
+		(start 227.693931 88.85)
+		(end 231.25 85.293931)
 		(width 0.4)
 		(layer "F.Cu")
